Commit message: som

File: workspaces/sim_ws/src/robot_sim/urdf/world/rubble/rubble.urdf (robot description, URDF)
Before this commit: robot wheeled_robot, 2 links, 1 joints
Links:
- link base_link: mass 7.3386e-05 -> 0.07338599999999999; geometry collision box size=0.03 0.03 0.03; visual box size=0.03 0.03 0.03

Commit message: Added cam test run script

File: workspaces/sim_ws/src/robot_sim/urdf/world/rubble/rubble.urdf (robot description, URDF)
Before this commit: robot wheeled_robot, 2 links, 1 joints
Links:
- link base_link: mass 0.07338599999999999 -> 0.5436; geometry collision box size=0.1 0.1 0.02; visual box size=0.1 0.1 0.02
